Commit message: Basic setup for the real robot stable, including all Dynamixel control and receiving camera input

File: ros2_ws/src/tidybot_description/urdf/tidybot_wx250s.urdf.xacro (robot description, xacro)
@@ -328,7 +328,7 @@
       <parent link="${prefix}_fingers_link"/>
       <child link="${prefix}_left_finger_link"/>
-      <origin xyz="0 0.015 0" rpy="0 0 0"/>
+      <origin xyz="0 0 0" rpy="0 0 0"/>
       <axis xyz="0 1 0"/>
-      <limit lower="-0.014" upper="0.022" effort="5" velocity="1"/>
+      <limit lower="0.015" upper="0.037" effort="5" velocity="1"/>
       <dynamics damping="0.1"/>
     </joint>
@@ -351,7 +351,7 @@
       <parent link="${prefix}_fingers_link"/>
       <child link="${prefix}_right_finger_link"/>
-      <origin xyz="0 -0.015 0" rpy="0 0 0"/>
+      <origin xyz="0 0 0" rpy="0 0 0"/>
       <axis xyz="0 -1 0"/>
-      <limit lower="-0.014" upper="0.022" effort="5" velocity="1"/>
+      <limit lower="0.015" upper="0.037" effort="5" velocity="1"/>
       <dynamics damping="0.1"/>
     </joint>

Commit message: Updated link names to use tf

File: ros2_ws/src/tidybot_description/urdf/tidybot_wx250s.urdf.xacro (robot description, xacro)
@@ -118,14 +118,15 @@
   </joint>
   <!-- Camera optical frames (Z forward, X right, Y down - standard ROS convention) -->
-  <link name="d435_color_optical_frame"/>
+  <!-- These frames are published by RealSense driver on real robot, but needed in URDF for simulation -->
+  <link name="camera_color_optical_frame"/>
   <joint name="camera_to_color_optical" type="fixed">
     <parent link="camera_link"/>
-    <child link="d435_color_optical_frame"/>
+    <child link="camera_color_optical_frame"/>
     <origin xyz="0 0 0" rpy="-1.5708 0 -1.5708"/>
   </joint>
-  <link name="d435_depth_optical_frame"/>
+  <link name="camera_depth_optical_frame"/>
   <joint name="camera_to_depth_optical" type="fixed">
     <parent link="camera_link"/>
-    <child link="d435_depth_optical_frame"/>
+    <child link="camera_depth_optical_frame"/>
     <origin xyz="0 0 0" rpy="-1.5708 0 -1.5708"/>
   </joint>
